File: esp.kicad_sch (KiCad schematic)
At the start: 119 parts, among them J1 Barrel_Jack, J11 Barrel_Jack, J12 Barrel_Jack, J13 Barrel_Jack, J14 Barrel_Jack, J2 8P8C_Shielded, J21 8P8C_Shielded, J27 Barrel_Jack, J3 Barrel_Jack, J38 8P8C_Shielded, J39 Barrel_Jack, J4 Barrel_Jack, J40 Barrel_Jack, J42 Barrel_Jack, J5 Barrel_Jack, J7 Barrel_Jack_MountingPin, K1 RT314A24, K5 RT314A24, K6 SRD-05VDC-SL-C, P1 Conn_WallPlug_Earth, Q3 MOSFET-NCHANNELSMD, Q4 MOSFET-NCHANNELSMD, Q5 MOSFET-NCHANNELSMD, Q6 NPN, SW1 SW_SPDT_MSM, U1 ESP32-S2-WROVER, U14 L298N, U15 PCF8574ATS, U16 L298N, U17 L298N, U18 NID30S48-24, U19 PCA9685PW, U2 TCA9548ARGER, U20 PCF8574ATS, U21 PC357_OPTO, U3 TCA9548ARGER, U4 BME280, U5 PCF8574ATS, U6 L298N, U7 OKI-78SR-12_1.0-W36H-C, U8 OKI-78SR-5_1.5-W36-C, U9 OKI-78SR-3.3_1.5-W36H-C

Commit message: fun
Connections:
- net TCA_2_SD7: now also J38.8
Other:
- sheet POE ports: added SDA; removed none
Changed lines of the file:
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@@
   (junction (at 247.65 332.74) (diameter 0) (color 0 0 0 0)
   )
+  (junction (at 454.66 231.14) (diameter 0) (color 0 0 0 0)
+  )
   (junction (at 259.08 312.42) (diameter 0) (color 0 0 0 0)
   )
@@
     (stroke (width 0) (type default))
   )
+  (wire (pts (xy 438.15 231.14) (xy 454.66 231.14))
+    (stroke (width 0) (type default))
+  )
   (wire (pts (xy 230.8951 327.66) (xy 236.22 327.66))
     (stroke (width 0) (type default))
@@
     (stroke (width 0) (type default))
   )
+  (wire (pts (xy 454.66 231.14) (xy 482.6 231.14))
+    (stroke (width 0) (type default))
+  )
   (wire (pts (xy 147.32 139.7) (xy 147.32 142.875))
     (stroke (width 0) (type solid))
@@
     (stroke (width 0.1524) (type solid))
   )
+  (wire (pts (xy 482.6 259.08) (xy 482.6 231.14))
+    (stroke (width 0) (type default))
+  )
   (wire (pts (xy 260.35 401.32) (xy 260.35 402.59))
     (stroke (width 0) (type default))
@@
     (stroke (width 0) (type default))
   )
+  (wire (pts (xy 499.11 259.08) (xy 482.6 259.08))
+    (stroke (width 0) (type default))
+  )
   (wire (pts (xy 486.41 360.68) (xy 486.41 284.48))
     (stroke (width 0) (type default))
@@
     )
   )
+  (global_label "TCA_2_SD7" (shape input) (at 454.66 231.14 0) (fields_autoplaced)
+    (effects (font (size 1.27 1.27)) (justify left))
+    (property "Intersheetrefs" "${INTERSHEET_REFS}" (at 467.8051 231.14 0)
+      (effects (font (size 1.27 1.27)) (justify left) hide)
+    )
+  )
   (global_label "PCF_3_GPIO_2" (shape input) (at 288.29 231.14 180) (fields_autoplaced)
     (effects (font (size 1.27 1.27)) (justify right))
@@
       (effects (font (size 1.27 1.27)) (justify left top))
     )
+    (pin "SDA" input (at 454.66 231.14 0)
+      (effects (font (size 1.27 1.27)) (justify right))
+    )
     (instances
