File: Barrel_Jack_Large_Motor.kicad_sch (KiCad schematic)
At the start: 32 parts, among them J15 Barrel_Jack, J16 Barrel_Jack, J17 Barrel_Jack, J18 Barrel_Jack, J19 Barrel_Jack, J20 Barrel_Jack, J36 Barrel_Jack, J37 Barrel_Jack, U10 PCF8574ATS, U27 L298N, U28 L298N, U29 L298N, U37 L298N, U38 PCF8574ATS, U39 PCA9685PW

Commit message: slimmed down and spread out pcb
Parts:
- removed C1: 220uF, symbol Device:C_Polarized_Small_US
- removed D1, D2, D3, D4, D5, D6, D7, D8: 1N4001, Diode_THT:D_DO-41_SOD81_P10.16mm_Horizontal, symbol Diode:1N4001
- removed F29, F30, F31, F32, F33, F34, F35, F36: Fuse, symbol Device:Fuse
- removed J15, J16, J17, J18, J19, J20, J36, J37: Barrel_Jack, symbol Connector:Barrel_Jack
- removed U10, U38: PCF8574ATS, Package_SO:SSOP-20_4.4x6.5mm_P0.65mm, symbol Interface_Expansion:PCF8574ATS
- removed U27, U28, U29, U37: L298N, Package_TO_SOT_THT:TO-220-15_P2.54x2.54mm_StaggerOdd_Lead4.58mm_Vertical, symbol Driver_Motor:L298N
- removed U39: PCA9685PW, Package_SO:TSSOP-28_4.4x9.7mm_P0.65mm, symbol Driver_LED:PCA9685PW
