File: I2C_POE.kicad_sch (KiCad schematic)
At the start: 6 parts, among them J22 8P8C_Shielded, J23 8P8C_Shielded, J24 8P8C_Shielded, J25 8P8C_Shielded, U11 PCA9548ADW

Commit message: slimmed down and spread out pcb
Parts:
- removed BT5: Battery, symbol Device:Battery
- removed J22, J23, J24, J25: 8P8C_Shielded, Connector_RJ:RJ45_HALO_HFJ11-x2450HRL_Horizontal, symbol Connector:8P8C_Shielded
- removed U11: PCA9548ADW, Package_SO:SOIC-24W_7.5x15.4mm_P1.27mm, symbol Interface_Expansion:PCA9548ADW
