File: POE.kicad_sch (KiCad schematic)
At the start: 0 parts

Commit message: fun
Parts:
- added J43: 8P8C_Shielded, Connector_RJ:RJ45_HALO_HFJ11-x2450HRL_Horizontal, symbol Connector:8P8C_Shielded
Connections:
- new net SDA: J43.8
Changed lines of the file:
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@@
 (kicad_sch (version 20230121) (generator eeschema)
   (paper "A4")
+  (hierarchical_label "SDA" (shape input) (at 173.99 46.99 0) (fields_autoplaced)
+    (effects (font (size 1.27 1.27)) (justify left))
+  )
+  (symbol (lib_id "Connector:8P8C_Shielded") (at 163.83 57.15 0) (unit 1)
+    (in_bom yes) (on_board yes) (dnp no) (fields_autoplaced)
+    (property "Reference" "J43" (at 163.83 39.37 0)
+      (effects (font (size 1.27 1.27)))
+    )
+    (property "Value" "8P8C_Shielded" (at 163.83 41.91 0)
+      (effects (font (size 1.27 1.27)))
+    )
+    (property "Footprint" "Connector_RJ:RJ45_HALO_HFJ11-x2450HRL_Horizontal" (at 163.83 56.515 90)
+      (effects (font (size 1.27 1.27)) hide)
+    )
+    (property "Datasheet" "~" (at 163.83 56.515 90)
+      (effects (font (size 1.27 1.27)) hide)
+    )
+    (pin "SH")
+    (pin "3")
+    (pin "4")
+    (pin "2")
+    (pin "8")
+    (pin "5")
+    (pin "7")
+    (pin "1")
+    (pin "6")
+    (instances
+      (project "esp"
+        (path "/dab6683c-420f-459a-bf9c-0c28b4b081e3/25046eec-894d-4c1f-90dd-413b7721facb"
+          (reference "J43") (unit 1)
+        )
+      )
+    )
+  )
 )

Commit message: slimmed down and spread out pcb
Parts:
- removed J43: 8P8C_Shielded, Connector_RJ:RJ45_HALO_HFJ11-x2450HRL_Horizontal, symbol Connector:8P8C_Shielded
Changed lines of the file:
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@@
 (kicad_sch (version 20230121) (generator eeschema)
   (paper "A4")
-  (hierarchical_label "SDA" (shape input) (at 173.99 46.99 0) (fields_autoplaced)
-    (effects (font (size 1.27 1.27)) (justify left))
-  )
-  (symbol (lib_id "Connector:8P8C_Shielded") (at 163.83 57.15 0) (unit 1)
-    (in_bom yes) (on_board yes) (dnp no) (fields_autoplaced)
-    (property "Reference" "J43" (at 163.83 39.37 0)
-      (effects (font (size 1.27 1.27)))
-    )
-    (property "Value" "8P8C_Shielded" (at 163.83 41.91 0)
-      (effects (font (size 1.27 1.27)))
-    )
-    (property "Footprint" "Connector_RJ:RJ45_HALO_HFJ11-x2450HRL_Horizontal" (at 163.83 56.515 90)
-      (effects (font (size 1.27 1.27)) hide)
-    )
-    (property "Datasheet" "~" (at 163.83 56.515 90)
-      (effects (font (size 1.27 1.27)) hide)
-    )
-    (pin "SH")
-    (pin "3")
-    (pin "4")
-    (pin "2")
-    (pin "8")
-    (pin "5")
-    (pin "7")
-    (pin "1")
-    (pin "6")
-    (instances
-      (project "esp"
-        (path "/dab6683c-420f-459a-bf9c-0c28b4b081e3/25046eec-894d-4c1f-90dd-413b7721facb"
-          (reference "J43") (unit 1)
-        )
-      )
-    )
-  )
 )
