File: Relay_Out.kicad_sch (KiCad schematic)
At the start: 0 parts

Commit message: some relay adjustments
Parts:
- added K10, K2, K3, K4, K8, K9: RT314A24, Relay_THT:Relay_1P1T_NO_10x24x18.8mm_Panasonic_ADW11xxxxW_THT, symbol Relay:RT314A24
- added U13: PCF8574ATS, Package_SO:SSOP-20_4.4x6.5mm_P0.65mm, symbol Interface_Expansion:PCF8574ATS
Changed lines of the file:
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@@
 (kicad_sch (version 20230121) (generator eeschema)
   (paper "A4")
+  (symbol (lib_id "Relay:RT314A24") (at 120.65 180.34 90) (unit 1)
+    (in_bom yes) (on_board yes) (dnp no) (fields_autoplaced)
+    (property "Reference" "K2" (at 119.38 168.91 0)
+      (effects (font (size 1.27 1.27)) (justify left))
+    )
+    (property "Value" "RT314A24" (at 121.92 168.91 0)
+      (effects (font (size 1.27 1.27)) (justify left))
+    )
+    (property "Footprint" "Relay_THT:Relay_1P1T_NO_10x24x18.8mm_Panasonic_ADW11xxxxW_THT" (at 121.92 140.97 0)
+      (effects (font (size 1.27 1.27)) hide)
+    )
+    (property "Datasheet" "https://www.te.com/commerce/DocumentDelivery/DDEController?Action=srchrtrv&DocNm=RT1_bistable&DocType=DS&DocLang=English" (at 120.65 180.34 0)
+      (effects (font (size 1.27 1.27)) hide)
+    )
+    (pin "11")
+    (pin "14")
+    (pin "12")
+    (pin "A1")
+    (pin "A2")
+    (instances
+      (project "esp"
+        (path "/dab6683c-420f-459a-bf9c-0c28b4b081e3/5a0a56ac-e74e-4f82-83ef-b10283bca7a0"
+          (reference "K2") (unit 1)
+        )
+      )
+    )
+  )
+  (symbol (lib_id "Relay:RT314A24") (at 121.92 115.57 90) (unit 1)
+    (in_bom yes) (on_board yes) (dnp no) (fields_autoplaced)
+    (property "Reference" "K4" (at 120.65 104.14 0)
+      (effects (font (size 1.27 1.27)) (justify left))
+    )
+    (property "Value" "RT314A24" (at 123.19 104.14 0)
+      (effects (font (size 1.27 1.27)) (justify left))
+    )
+    (property "Footprint" "Relay_THT:Relay_1P1T_NO_10x24x18.8mm_Panasonic_ADW11xxxxW_THT" (at 123.19 76.2 0)
+      (effects (font (size 1.27 1.27)) hide)
+    )
+    (property "Datasheet" "https://www.te.com/commerce/DocumentDelivery/DDEController?Action=srchrtrv&DocNm=RT1_bistable&DocType=DS&DocLang=English" (at 121.92 115.57 0)
+      (effects (font (size 1.27 1.27)) hide)
+    )
+    (pin "11")
+    (pin "14")
+    (pin "12")
+    (pin "A1")
+    (pin "A2")
+    (instances
+      (project "esp"
+        (path "/dab6683c-420f-459a-bf9c-0c28b4b081e3/5a0a56ac-e74e-4f82-83ef-b10283bca7a0"
+          (reference "K4") (unit 1)
+        )
+      )
+    )
+  )
+  (symbol (lib_id "Interface_Expansion:PCF8574ATS") (at 236.22 96.52 180) (unit 1)
+    (in_bom yes) (on_board yes) (dnp no) (fields_autoplaced)
+    (property "Reference" "U13" (at 236.5659 76.2 0)
+      (effects (font (size 1.27 1.27)) (justify right))
+    )
+    (property "Value" "PCF8574ATS" (at 236.5659 78.74 0)
+      (effects (font (size 1.27 1.27)) (justify right))
+    )
+    (property "Footprint" "Package_SO:SSOP-20_4.4x6.5mm_P0.65mm" (at 236.22 96.52 0)
+      (effects (font (size 1.27 1.27)) hide)
+    )
+    (property "Datasheet" "http://www.nxp.com/docs/en/data-sheet/PCF8574_PCF8574A.pdf" (at 236.22 96.52 0)
+      (effects (font (size 1.27 1.27)) hide)
+    )
+    (pin "8")
+    (pin "5")
+    (pin "3")
+    (pin "4")
+    (pin "13")
+    (pin "6")
+    (pin "10")
+    (pin "11")
+    (pin "18")
+    (pin "7")
+    (pin "17")
+    (pin "15")
+    (pin "20")
+    (pin "9")
+    (pin "2")
+    (pin "12")
+    (pin "1")
+    (pin "19")
+    (pin "16")
+    (pin "14")
+    (instances
+      (project "esp"
+        (path "/dab6683c-420f-459a-bf9c-0c28b4b081e3/5a0a56ac-e74e-4f82-83ef-b10283bca7a0"
+          (reference "U13") (unit 1)
+        )
+      )
+    )
+  )
+  (symbol (lib_id "Relay:RT314A24") (at 146.05 34.29 90) (unit 1)
+    (in_bom yes) (on_board yes) (dnp no) (fields_autoplaced)
+    (property "Reference" "K10" (at 144.78 22.86 0)
+      (effects (font (size 1.27 1.27)) (justify left))
+    )
+    (property "Value" "RT314A24" (at 147.32 22.86 0)
+      (effects (font (size 1.27 1.27)) (justify left))
+    )
+    (property "Footprint" "Relay_THT:Relay_1P1T_NO_10x24x18.8mm_Panasonic_ADW11xxxxW_THT" (at 147.32 -5.08 0)
+      (effects (font (size 1.27 1.27)) hide)
+    )
+    (property "Datasheet" "https://www.te.com/commerce/DocumentDelivery/DDEController?Action=srchrtrv&DocNm=RT1_bistable&DocType=DS&DocLang=English" (at 146.05 34.29 0)
+      (effects (font (size 1.27 1.27)) hide)
+    )
+    (pin "11")
+    (pin "14")
+    (pin "12")
+    (pin "A1")
+    (pin "A2")
+    (instances
+      (project "esp"
+        (path "/dab6683c-420f-459a-bf9c-0c28b4b081e3/5a0a56ac-e74e-4f82-83ef-b10283bca7a0"
+          (reference "K10") (unit 1)
+        )
+      )
+    )
+  )
+  (symbol (lib_id "Relay:RT314A24") (at 145.415 66.675 90) (unit 1)
+    (in_bom yes) (on_board yes) (dnp no) (fields_autoplaced)
+    (property "Reference" "K9" (at 144.145 55.245 0)
+      (effects (font (size 1.27 1.27)) (justify left))
+    )
+    (property "Value" "RT314A24" (at 146.685 55.245 0)
+      (effects (font (size 1.27 1.27)) (justify left))
+    )
+    (property "Footprint" "Relay_THT:Relay_1P1T_NO_10x24x18.8mm_Panasonic_ADW11xxxxW_THT" (at 146.685 27.305 0)
+      (effects (font (size 1.27 1.27)) hide)
+    )
+    (property "Datasheet" "https://www.te.com/commerce/DocumentDelivery/DDEController?Action=srchrtrv&DocNm=RT1_bistable&DocType=DS&DocLang=English" (at 145.415 66.675 0)
+      (effects (font (size 1.27 1.27)) hide)
+    )
+    (pin "11")
+    (pin "14")
+    (pin "12")
+    (pin "A1")
+    (pin "A2")
+    (instances
+      (project "esp"
+        (path "/dab6683c-420f-459a-bf9c-0c28b4b081e3/5a0a56ac-e74e-4f82-83ef-b10283bca7a0"
+          (reference "K9") (unit 1)
+        )
+      )
+    )
+  )
+  (symbol (lib_id "Relay:RT314A24") (at 121.285 147.955 90) (unit 1)
+    (in_bom yes) (on_board yes) (dnp no) (fields_autoplaced)
+    (property "Reference" "K3" (at 120.015 136.525 0)
+      (effects (font (size 1.27 1.27)) (justify left))
+    )
+    (property "Value" "RT314A24" (at 122.555 136.525 0)
+      (effects (font (size 1.27 1.27)) (justify left))
+    )
+    (property "Footprint" "Relay_THT:Relay_1P1T_NO_10x24x18.8mm_Panasonic_ADW11xxxxW_THT" (at 122.555 108.585 0)
+      (effects (font (size 1.27 1.27)) hide)
+    )
+    (property "Datasheet" "https://www.te.com/commerce/DocumentDelivery/DDEController?Action=srchrtrv&DocNm=RT1_bistable&DocType=DS&DocLang=English" (at 121.285 147.955 0)
+      (effects (font (size 1.27 1.27)) hide)
+    )
+    (pin "11")
+    (pin "14")
+    (pin "12")
+    (pin "A1")
+    (pin "A2")
+    (instances
+      (project "esp"
+        (path "/dab6683c-420f-459a-bf9c-0c28b4b081e3/5a0a56ac-e74e-4f82-83ef-b10283bca7a0"
+          (reference "K3") (unit 1)
+        )
+      )
+    )
+  )
+  (symbol (lib_id "Relay:RT314A24") (at 144.78 99.06 90) (unit 1)
+    (in_bom yes) (on_board yes) (dnp no) (fields_autoplaced)
+    (property "Reference" "K8" (at 143.51 87.63 0)
+      (effects (font (size 1.27 1.27)) (justify left))
+    )
+    (property "Value" "RT314A24" (at 146.05 87.63 0)
+      (effects (font (size 1.27 1.27)) (justify left))
+    )
+    (property "Footprint" "Relay_THT:Relay_1P1T_NO_10x24x18.8mm_Panasonic_ADW11xxxxW_THT" (at 146.05 59.69 0)
+      (effects (font (size 1.27 1.27)) hide)
+    )
+    (property "Datasheet" "https://www.te.com/commerce/DocumentDelivery/DDEController?Action=srchrtrv&DocNm=RT1_bistable&DocType=DS&DocLang=English" (at 144.78 99.06 0)
+      (effects (font (size 1.27 1.27)) hide)
+    )
+    (pin "11")
+    (pin "14")
+    (pin "12")
+    (pin "A1")
+    (pin "A2")
+    (instances
+      (project "esp"
+        (path "/dab6683c-420f-459a-bf9c-0c28b4b081e3/5a0a56ac-e74e-4f82-83ef-b10283bca7a0"
+          (reference "K8") (unit 1)
+        )
+      )
+    )
+  )
 )

Commit message: slimmed down and spread out pcb
Parts:
- removed K10, K2, K3, K4, K8, K9: RT314A24, Relay_THT:Relay_1P1T_NO_10x24x18.8mm_Panasonic_ADW11xxxxW_THT, symbol Relay:RT314A24
- removed U13: PCF8574ATS, Package_SO:SSOP-20_4.4x6.5mm_P0.65mm, symbol Interface_Expansion:PCF8574ATS
Changed lines of the file:
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@@
 (kicad_sch (version 20230121) (generator eeschema)
   (paper "A4")
-  (symbol (lib_id "Relay:RT314A24") (at 120.65 180.34 90) (unit 1)
-    (in_bom yes) (on_board yes) (dnp no) (fields_autoplaced)
-    (property "Reference" "K2" (at 119.38 168.91 0)
-      (effects (font (size 1.27 1.27)) (justify left))
-    )
-    (property "Value" "RT314A24" (at 121.92 168.91 0)
-      (effects (font (size 1.27 1.27)) (justify left))
-    )
-    (property "Footprint" "Relay_THT:Relay_1P1T_NO_10x24x18.8mm_Panasonic_ADW11xxxxW_THT" (at 121.92 140.97 0)
-      (effects (font (size 1.27 1.27)) hide)
-    )
-    (property "Datasheet" "https://www.te.com/commerce/DocumentDelivery/DDEController?Action=srchrtrv&DocNm=RT1_bistable&DocType=DS&DocLang=English" (at 120.65 180.34 0)
-      (effects (font (size 1.27 1.27)) hide)
-    )
-    (pin "11")
-    (pin "14")
-    (pin "12")
-    (pin "A1")
-    (pin "A2")
-    (instances
-      (project "esp"
-        (path "/dab6683c-420f-459a-bf9c-0c28b4b081e3/5a0a56ac-e74e-4f82-83ef-b10283bca7a0"
-          (reference "K2") (unit 1)
-        )
-      )
-    )
-  )
-  (symbol (lib_id "Relay:RT314A24") (at 121.92 115.57 90) (unit 1)
-    (in_bom yes) (on_board yes) (dnp no) (fields_autoplaced)
-    (property "Reference" "K4" (at 120.65 104.14 0)
-      (effects (font (size 1.27 1.27)) (justify left))
-    )
-    (property "Value" "RT314A24" (at 123.19 104.14 0)
-      (effects (font (size 1.27 1.27)) (justify left))
-    )
-    (property "Footprint" "Relay_THT:Relay_1P1T_NO_10x24x18.8mm_Panasonic_ADW11xxxxW_THT" (at 123.19 76.2 0)
-      (effects (font (size 1.27 1.27)) hide)
-    )
-    (property "Datasheet" "https://www.te.com/commerce/DocumentDelivery/DDEController?Action=srchrtrv&DocNm=RT1_bistable&DocType=DS&DocLang=English" (at 121.92 115.57 0)
-      (effects (font (size 1.27 1.27)) hide)
-    )
-    (pin "11")
-    (pin "14")
-    (pin "12")
-    (pin "A1")
-    (pin "A2")
-    (instances
-      (project "esp"
-        (path "/dab6683c-420f-459a-bf9c-0c28b4b081e3/5a0a56ac-e74e-4f82-83ef-b10283bca7a0"
-          (reference "K4") (unit 1)
-        )
-      )
-    )
-  )
-  (symbol (lib_id "Interface_Expansion:PCF8574ATS") (at 236.22 96.52 180) (unit 1)
-    (in_bom yes) (on_board yes) (dnp no) (fields_autoplaced)
-    (property "Reference" "U13" (at 236.5659 76.2 0)
-      (effects (font (size 1.27 1.27)) (justify right))
-    )
-    (property "Value" "PCF8574ATS" (at 236.5659 78.74 0)
-      (effects (font (size 1.27 1.27)) (justify right))
-    )
-    (property "Footprint" "Package_SO:SSOP-20_4.4x6.5mm_P0.65mm" (at 236.22 96.52 0)
-      (effects (font (size 1.27 1.27)) hide)
-    )
-    (property "Datasheet" "http://www.nxp.com/docs/en/data-sheet/PCF8574_PCF8574A.pdf" (at 236.22 96.52 0)
-      (effects (font (size 1.27 1.27)) hide)
-    )
-    (pin "8")
-    (pin "5")
-    (pin "3")
-    (pin "4")
-    (pin "13")
-    (pin "6")
-    (pin "10")
-    (pin "11")
-    (pin "18")
-    (pin "7")
-    (pin "17")
-    (pin "15")
-    (pin "20")
-    (pin "9")
-    (pin "2")
-    (pin "12")
-    (pin "1")
-    (pin "19")
-    (pin "16")
-    (pin "14")
-    (instances
-      (project "esp"
-        (path "/dab6683c-420f-459a-bf9c-0c28b4b081e3/5a0a56ac-e74e-4f82-83ef-b10283bca7a0"
-          (reference "U13") (unit 1)
-        )
-      )
-    )
-  )
-  (symbol (lib_id "Relay:RT314A24") (at 146.05 34.29 90) (unit 1)
-    (in_bom yes) (on_board yes) (dnp no) (fields_autoplaced)
-    (property "Reference" "K10" (at 144.78 22.86 0)
-      (effects (font (size 1.27 1.27)) (justify left))
-    )
-    (property "Value" "RT314A24" (at 147.32 22.86 0)
-      (effects (font (size 1.27 1.27)) (justify left))
-    )
-    (property "Footprint" "Relay_THT:Relay_1P1T_NO_10x24x18.8mm_Panasonic_ADW11xxxxW_THT" (at 147.32 -5.08 0)
-      (effects (font (size 1.27 1.27)) hide)
-    )
-    (property "Datasheet" "https://www.te.com/commerce/DocumentDelivery/DDEController?Action=srchrtrv&DocNm=RT1_bistable&DocType=DS&DocLang=English" (at 146.05 34.29 0)
-      (effects (font (size 1.27 1.27)) hide)
-    )
-    (pin "11")
-    (pin "14")
-    (pin "12")
-    (pin "A1")
-    (pin "A2")
-    (instances
-      (project "esp"
-        (path "/dab6683c-420f-459a-bf9c-0c28b4b081e3/5a0a56ac-e74e-4f82-83ef-b10283bca7a0"
-          (reference "K10") (unit 1)
-        )
-      )
-    )
-  )
-  (symbol (lib_id "Relay:RT314A24") (at 145.415 66.675 90) (unit 1)
-    (in_bom yes) (on_board yes) (dnp no) (fields_autoplaced)
-    (property "Reference" "K9" (at 144.145 55.245 0)
-      (effects (font (size 1.27 1.27)) (justify left))
-    )
-    (property "Value" "RT314A24" (at 146.685 55.245 0)
-      (effects (font (size 1.27 1.27)) (justify left))
-    )
-    (property "Footprint" "Relay_THT:Relay_1P1T_NO_10x24x18.8mm_Panasonic_ADW11xxxxW_THT" (at 146.685 27.305 0)
-      (effects (font (size 1.27 1.27)) hide)
-    )
-    (property "Datasheet" "https://www.te.com/commerce/DocumentDelivery/DDEController?Action=srchrtrv&DocNm=RT1_bistable&DocType=DS&DocLang=English" (at 145.415 66.675 0)
-      (effects (font (size 1.27 1.27)) hide)
-    )
-    (pin "11")
-    (pin "14")
-    (pin "12")
-    (pin "A1")
-    (pin "A2")
-    (instances
-      (project "esp"
-        (path "/dab6683c-420f-459a-bf9c-0c28b4b081e3/5a0a56ac-e74e-4f82-83ef-b10283bca7a0"
-          (reference "K9") (unit 1)
-        )
-      )
-    )
-  )
-  (symbol (lib_id "Relay:RT314A24") (at 121.285 147.955 90) (unit 1)
-    (in_bom yes) (on_board yes) (dnp no) (fields_autoplaced)
-    (property "Reference" "K3" (at 120.015 136.525 0)
-      (effects (font (size 1.27 1.27)) (justify left))
-    )
-    (property "Value" "RT314A24" (at 122.555 136.525 0)
-      (effects (font (size 1.27 1.27)) (justify left))
-    )
-    (property "Footprint" "Relay_THT:Relay_1P1T_NO_10x24x18.8mm_Panasonic_ADW11xxxxW_THT" (at 122.555 108.585 0)
-      (effects (font (size 1.27 1.27)) hide)
-    )
-    (property "Datasheet" "https://www.te.com/commerce/DocumentDelivery/DDEController?Action=srchrtrv&DocNm=RT1_bistable&DocType=DS&DocLang=English" (at 121.285 147.955 0)
-      (effects (font (size 1.27 1.27)) hide)
-    )
-    (pin "11")
-    (pin "14")
-    (pin "12")
-    (pin "A1")
-    (pin "A2")
-    (instances
-      (project "esp"
-        (path "/dab6683c-420f-459a-bf9c-0c28b4b081e3/5a0a56ac-e74e-4f82-83ef-b10283bca7a0"
-          (reference "K3") (unit 1)
-        )
-      )
-    )
-  )
-  (symbol (lib_id "Relay:RT314A24") (at 144.78 99.06 90) (unit 1)
-    (in_bom yes) (on_board yes) (dnp no) (fields_autoplaced)
-    (property "Reference" "K8" (at 143.51 87.63 0)
-      (effects (font (size 1.27 1.27)) (justify left))
-    )
-    (property "Value" "RT314A24" (at 146.05 87.63 0)
-      (effects (font (size 1.27 1.27)) (justify left))
-    )
-    (property "Footprint" "Relay_THT:Relay_1P1T_NO_10x24x18.8mm_Panasonic_ADW11xxxxW_THT" (at 146.05 59.69 0)
-      (effects (font (size 1.27 1.27)) hide)
-    )
-    (property "Datasheet" "https://www.te.com/commerce/DocumentDelivery/DDEController?Action=srchrtrv&DocNm=RT1_bistable&DocType=DS&DocLang=English" (at 144.78 99.06 0)
-      (effects (font (size 1.27 1.27)) hide)
-    )
-    (pin "11")
-    (pin "14")
-    (pin "12")
-    (pin "A1")
-    (pin "A2")
-    (instances
-      (project "esp"
-        (path "/dab6683c-420f-459a-bf9c-0c28b4b081e3/5a0a56ac-e74e-4f82-83ef-b10283bca7a0"
-          (reference "K8") (unit 1)
-        )
-      )
-    )
-  )
 )
